File: 2019-01 Temperature Sensor.kicad_pcb (KiCad board)
At the start: 2 copper layers, 6 parts, among them J1 Conn_01x03, U1 MCP9701AT

Commit message: Completed layout of the board.
Parts:
- added H1: MountingHole, 0_Mechanical:MountingHole_3.2mm_M3, F.Cu at (117.0, 92.5)
- added REF**: OSHW-Logo_5.7x6mm_SilkScreen, Symbol:OSHW-Logo_5.7x6mm_SilkScreen, F.Cu at (126.5, 88.3)
- moved J1 20.9 mm to (109.1, 92.5)
- moved U1 19.3 mm to (126.9, 96.2)
- moved R2 19.0 mm to (123.2, 95.1)
- moved C2 16.6 mm to (123.2, 97.2), turned to 0 degrees
- moved C1 14.7 mm to (126.8, 92.9), turned to 0 degrees
- moved R1 14.0 mm to (123.2, 92.9)
Routing:
- net Net-(C2-Pad1): track 0.00 -> 21.2 mm
- net Net-(J1-Pad1): track 0.00 -> 20.6 mm
- net Net-(C1-Pad1): track 0.00 -> 5.86 mm
- net Net-(R2-Pad1): track 0.00 -> 2.01 mm
- added copper zone on F.Cu, net GND
Other:
- board outline added: 30 x 15 mm
- net class Default: clearance 0.2 -> 0.3; trace_width 0.25 -> 0.4; via_dia 0.8 -> 0.6; via_drill 0.4 -> 0.3
- rule pad_to_mask_clearance: 0.051 -> 0.0508
- rule solder_mask_min_width: 0.25 -> 0.15
- rule trace_clearance: 0.2 -> 0.3
- board text added: "2019-01-Temperature-Sensor"
- board text added: "Copyright © 2019 Marco Chiu"
